Commit message: mesh

File: src/robot_sim/urdf/model.urdf (robot description, URDF)
Before this commit: robot wheelchair, 18 links, 17 joints
Links:
- removed link base_footprint
- removed link base_link
- removed link front_left_swivel
- removed link front_left_wheel
- removed link front_right_swivel
- removed link front_right_wheel
- removed link imu_link
- removed link left_bar
- removed link left_main_wheel
- removed link left_scanner
- removed link legs
- removed link rear_left_swivel
- removed link rear_left_wheel
- removed link rear_right_swivel
- removed link rear_right_wheel
- removed link right_bar
- removed link right_main_wheel
- removed link right_scanner
- added link chassis, mass 10.0; collision box size=0.406054 0.406054 0.10; visual box size=0.01 0.01 0.10
- added link left_wheel, mass 0.5; collision cylinder length=0.0356884 radius=0.201784; visual mesh filename=package://robot_sim/meshes/wheelchair_wheel.stl scale=0.01 0.01 0.01
- added link right_wheel, mass 0.5; collision cylinder length=0.0356884 radius=0.201784; visual mesh filename=package://robot_sim/meshes/wheelchair_wheel.stl scale=0.01 0.01 0.01
Joints:
- removed joint base_footprint_joint
- removed joint front_left_swivel_joint
- removed joint front_left_wheel_joint
- removed joint front_right_swivel_joint
- removed joint front_right_wheel_joint
- removed joint imu_joint
- removed joint left_bar_joint
- removed joint left_main_wheel_joint
- removed joint left_scanner_joint
- removed joint legs_joint
- removed joint rear_left_swivel_joint
- removed joint rear_left_wheel_joint
- removed joint rear_right_swivel_joint
- removed joint rear_right_wheel_joint
- removed joint right_bar_joint
- removed joint right_main_wheel_joint
- removed joint right_scanner_joint
- added joint left_wheel_hinge: type continuous, parent chassis, child left_wheel, origin xyz=0 0.19 0.201784 rpy=0 0 0, axis 0 1 0, limit effort=100 velocity=100
- added joint right_wheel_hinge: type continuous, parent chassis, child right_wheel, origin xyz=0 -0.19 0.201784 rpy=0 0 0, axis 0 1 0, limit effort=100 velocity=100

File: src/robot_sim/urdf/robot.xacro (robot description, xacro)
@@ -1,129 +1,66 @@
 <?xml version='1.0'?>
-<robot name="robot" xmlns:xacro="http://www.ros.org/wiki/xacro">
-  <link name='chassis'>
+<robot name="wheelchair" xmlns:xacro="http://www.ros.org/wiki/xacro" >
+  <xacro:property name="cameraSize" value="0.05"/>
+  <xacro:property name="cameraMass" value="0.1"/>
+  <xacro:property name="PI" value="3.14" />
+  <xacro:property name="PI_Half" value="1.5707" />
+  <xacro:property name="chair_width" value="0.643" /> <!-- From front wheel right joint to front wheel left joint -->
+  <xacro:property name="chair_length" value="0.812" /> <!-- From front wheel joint to back wheel joint -->
+  <xacro:property name="chair_height" value="1.191" /> <!-- From front wheel joint to head rest -->
+  <xacro:property name="chair_weight" value="10.0" />
+  <xacro:property name="legs_width" value="0.4064" />
+  <xacro:property name="legs_length" value="0.4064" />
+  <xacro:property name="legs_height" value="0.4064" />
+  <xacro:property name="legs_weight" value="2.0" />
+  <xacro:property name="main_wheel_length" value="0.0356884" />
+  <xacro:property name="main_wheel_radius" value="0.201784" />
+  <xacro:property name="main_wheel_weight" value="3.0" />
+  <xacro:property name="small_wheel_radius" value="0.068" />
+  <xacro:property name="small_wheel_length" value="0.032" />
+  <xacro:property name="small_wheel_weight" value="1.0" />
+  <xacro:include filename="$(find robot_sim)/urdf/materials.xacro" />
+  <xacro:include filename="$(find robot_sim)/urdf/macros.xacro" />
+  <link name='base_chassis'>
     <pose>0 0 0.201784 0 0 0</pose>
     <inertial>
       <mass value="10.0"/>
       <origin xyz="0 0 0.201784" rpy=" 0 0 0"/>
-      <inertia
-          ixx="1.0" ixy="0" ixz="0"
-          iyy="1.0" iyz="0"
-          izz="1.0"
-      />
+      <box_inertia m="2" x="0.01" y="0.01" z ="0.406054" />
     </inertial>
     <collision name='collision'>
       <geometry>
-        <box size="0.406054 0.406054 0.10"/>
+        <box size="0.01 0.406054 0.01"/>
       </geometry>
     </collision>
-    <visual name='chair'>
+    <visual>
       <origin xyz="0 0 0" rpy="0 0 -3.14"/>
       <geometry>
-         <!-- <box size="0.40 0.35  0.1"/>  -->
-        <mesh filename="package://robot_sim/meshes/wheelchair_chasis.stl" scale="0.01 0.01 0.01"/>
+         <mesh filename="package://robot_sim/meshes/wheelchair_chasis.stl" scale="0.01 0.01 0.01"/>
       </geometry>
-    </visual>
-    <!--
-    <visual name='os1'>
-      <origin xyz="0 0 0.40605" rpy=" 0 0 0"/>
-      <geometry>
-        <box size="0.016 0.016 0.40605"/>
-      </geometry>
-    </visual>
-    <visual name='osnova.001'>
-      <origin xyz="0.217474 0.159666 0.166384" rpy="1.5707 0 1.5707"/>
-      <geometry>
-        <box size="0.015709 0.015709 0.310168"/>
-      </geometry>
-    </visual>
+  </visual>
+  <visual>
+    <origin xyz="0 0 0.201784" rpy="0 0 0"/>
+    <geometry>
+      <box size="0.01 0.406054 0.01"/>
+    </geometry>
+</visual>
+</link>
+  <!--
+  <chassis name="base" xyz="0 0 ${main_wheel_radius}" rpy="0 0 0" m="2" chassisLength="0.01" chassisWidth="${2*main_wheel_radius}" chassisHeight="0.01"/>
 -->
-   <!--
-    <collision name='caster_collision'>
-      <origin xyz="0.406054 0 0.201784" rpy=" 0 0 0"/>
-      <geometry>
-        <sphere radius="0.201784"/>
-      </geometry>
-      <surface>
-        <friction>
-          <ode>
-            <mu>0</mu>
-            <mu2>0</mu2>
-            <slip1>1.0</slip1>
-            <slip2>1.0</slip2>
-          </ode>
-        </friction>
-      </surface>
-    </collision>
-    <visual name='caster_visual'>
-      <origin xyz="0.406054/2 0 0.201784" rpy=" 0 0 0"/>
-      <geometry>
-        <sphere radius="0.201784"/>
-      </geometry>
-    </visual>-->
-  </link>
-  <link name="left_wheel">
-    <collision name="collision">
-      <origin xyz="0 0 0" rpy="0 1.5707 1.5707"/>
-      <geometry>
-         <cylinder radius="0.201784" length="0.0356884"/>
-      </geometry>
-    </collision>
-    <visual name="left_wheel_visual">
-      <origin xyz="0 0 0" rpy="0 1.5707 1.5707"/>
-      <geometry>
-        <mesh filename="package://robot_sim/meshes/wheelchair_wheel.stl" scale="0.01 0.01 0.01"/>
-        <!-- <cylinder radius="0.201784" length="0.0356884"/> -->
-      </geometry>
-    </visual>
-    <inertial>
-      <origin xyz="0 0 0.201784" rpy="0 1.5707 1.5707"/>
-      <mass value="0.5"/>
-      <cylinder_inertia m="0.5" r="0.201784" h="0.0356884"/>
-      <inertia
-        ixx="0.1" ixy="0.0" ixz="0.0"
-        iyy="0.1" iyz="0.0"
-        izz="0.1"/>
-    </inertial>
-  </link>
-  <link name="right_wheel">
-    <collision name="collision">
-      <origin xyz="0 0 0" rpy="0 1.5707 -1.5707"/>
-      <geometry>
-        <cylinder radius="0.201784" length="0.0356884"/>
-    </geometry>
-    </collision>
-    <visual name="right_wheel_visual">
-      <origin xyz="0 0 0" rpy="0 1.5707 -1.5707"/>
-      <geometry>
-          <!-- <cylinder radius="0.201784" length="0.0356884"/> -->
-        <mesh filename="package://robot_sim/meshes/wheelchair_wheel.stl" scale="0.01 0.01 0.01"/>
-      </geometry>
-    </visual>
-    <inertial>
-      <origin xyz="0 0 0.201784" rpy="0 1.5707 1.5707"/>
-      <mass value="0.5"/>
-      <cylinder_inertia m="0.5" r="0.201784" h="0.0356884"/>
-      <inertia
-        ixx="0.1" ixy="0.0" ixz="0.0"
-        iyy="0.1" iyz="0.0"
-        izz="0.1"/>
-    </inertial>
-  </link>
-  <joint type="continuous" name="left_wheel_hinge">
-    <origin xyz="0 0.19 0.201784" rpy="0 0 0"/>
-    <child link="left_wheel"/>
-    <parent link="chassis"/>
-    <axis xyz="0 1 0" rpy="0 0 0"/>
-    <limit effort="100" velocity="100"/>
-    <joint_properties damping="0.0" friction="0.0"/>
-  </joint>
-  <joint type="continuous" name="right_wheel_hinge">
-    <origin xyz="0 -0.19 0.201784" rpy="0 0 0"/>
-    <child link="right_wheel"/>
-    <parent link="chassis"/>
-    <axis xyz="0 1 0" rpy="0 0 0"/>
-    <limit effort="100" velocity="100"/>
-    <joint_properties damping="0.0" friction="0.0"/>
-  </joint>
+  <chassis name="os" xyz="${main_wheel_radius} 0.01 0.01" rpy="0 0 0" m="2" chassisLength="${2*main_wheel_radius}" chassisWidth="0.01" chassisHeight="0.01"/>
+  <link_joint parent="base_chassis" child ="os_chassis" xyz="0 0 ${main_wheel_radius}" rpy="0 0 0" />
+  <chassis name="os1" xyz="${main_wheel_radius} 0 0" rpy="0 0 0" m="2" chassisLength="0.01" chassisWidth="${2*main_wheel_radius - 0.2}" chassisHeight="0.01"/>
+  <link_joint parent="os_chassis" child ="os1_chassis" xyz="${main_wheel_radius} 0 0" rpy="0 0 0" />
+  <chassis name="os2" xyz="0 0 ${-main_wheel_radius/2}" rpy="0 0 0" m="2" chassisLength="0.01" chassisWidth="0.01" chassisHeight="${main_wheel_radius}"/>
+  <link_joint parent="os1_chassis" child ="os2_chassis" xyz="${main_wheel_radius} ${main_wheel_radius/2} 0" rpy="0 0 0" />
+  <chassis name="os3" xyz="0 0 ${-main_wheel_radius/2}" rpy="0 0 0" m="2" chassisLength="0.01" chassisWidth="0.01" chassisHeight="${main_wheel_radius}"/>
+  <link_joint parent="os1_chassis" child ="os3_chassis" xyz="${main_wheel_radius} ${-main_wheel_radius/2} 0" rpy="0 0 0" />
+  <wheel  lr="l" tY="0.02" xyz=" 0 0 ${main_wheel_radius}" rpy="${-pi/2} 0 0" wheelWidth="${main_wheel_length}" wheelRadius="${main_wheel_radius}" wheelMass="${main_wheel_weight}" meshFile="wheelchair_wheel"/>
+  <wheel_joint parent="base_chassis" child ="l_wheel" xyz="0 ${main_wheel_radius} 0" rpy="0 0 0" />
+  <wheel  lr="r" tY="0.02" xyz=" 0 0 ${main_wheel_radius}" rpy="${pi/2} 0 0" wheelWidth="${main_wheel_length}" wheelRadius="${main_wheel_radius}" wheelMass="${main_wheel_weight}" meshFile="wheelchair_wheel"/>
+  <wheel_joint parent="base_chassis" child ="r_wheel" xyz="0 ${-main_wheel_radius} 0" rpy="0 0 0" />
+  <wheel  lr="lf" tY="0.001" xyz=" 0 0 0" rpy="${pi/2} 0 0" wheelWidth="${small_wheel_length}" wheelRadius="${small_wheel_radius}" wheelMass="${small_wheel_weight}" meshFile="wheelchair_wheel_front"/>
+  <wheel_joint parent="os2_chassis" child ="lf_wheel" xyz="${small_wheel_radius} ${small_wheel_radius} -${small_wheel_radius}" rpy="0 0 0" />
   <gazebo>
     <plugin name="differential_drive_controller" filename="libgazebo_ros_diff_drive.so">
