Commit message: Update macros.xacro

File: src/robot_sim/urdf/macros.xacro (robot description, xacro)
@@ -52,5 +52,5 @@
       </visual>
       <inertial name="${lr}_wheel_visual_intertial">
-        <origin xyz="0 0 0" rpy="0 ${pi/2} ${pi/2}" />
+        <origin xyz="${xyz}" rpy="0 ${pi/2} ${pi/2}" />
         <mass value="${wheelMass}"/>
         <cylinder_inertia m="${wheelMass}" r="${wheelRadius}" h="${wheelWidth}"/>
